File: KiCad/Wubbo.kicad_sch (KiCad schematic)
At the start: 46 parts, among them J1 USB_C_Receptacle, J2 SWD, J3 USB, J4 JST-BATT, J5 USB, Q1 AO3407, Q2 AO3407, SW1 Choc, SW10 Choc, SW11 Choc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

Commit message: Various modifications to make it 38 keys
Parts:
- added SW18, SW19: Choc, kiboard_cache:PG13500-reversible, symbol Switch:SW_Push
- J1: footprint USB-C-12-Pin-MidMount -> footprints:USB-C-12-Pin-MidMount
Connections:
- net unconnected-(U1-P0.12) is gone; now on net SW3: U1.17 (P0.12)
- net unconnected-(U1-P0.19) is gone; now on net SW4: U1.20 (P0.19)
- net GND: now also SW18.2, SW19.2
- net SW1: now also U1.5 (P1.15); no longer U1.4 (P1.13)
- net SW10: now also U1.8 (P0.28); no longer U1.26 (P0.22)
- net SW12: now also U1.34 (P1.06); no longer U1.5 (P1.15)
- net SW13: now also U1.33 (P1.04); no longer U1.34 (P1.06)
- net SW14: now also U1.30 (P1.02); no longer U1.33 (P1.04)
- net SW15: now also U1.29 (P1.01); no longer U1.30 (P1.02)
- net SW16: now also U1.4 (P1.13); no longer U1.3 (P1.10)
- net SW17: now also U1.3 (P1.10); no longer U1.2 (P1.11)
- net SW2: now also U1.10 (P0.30); no longer U1.8 (P0.28)
- net SW3: no longer U1.9 (P0.29)
- net SW4: no longer U1.10 (P0.30)
- net SW7: now also U1.28 (P1.03); no longer U1.29 (P1.01)
- net SW8: now also U1.27 (P1.00); no longer U1.28 (P1.03)
- net SW9: now also U1.26 (P0.22); no longer U1.27 (P1.00)
- new net SW18: SW18.1, U1.2 (P1.11)
- new net SW19: SW19.1, U1.9 (P0.29)
Other:
- moved on the sheet: SW1, SW11, SW6
